Commit message: stable version by tutroial of (7)

File: my_robo/my_robo_description/my_robo_tof.urdf (robot description, URDF)
Before this commit: robot my_robo, 6 links, 5 joints
Links:
- removed link hokuyo_link
- added link pico_flexx_depth_frame
- added link pico_flexx_link, mass 1; collision box size=0.007 0.066 0.016; visual box size=0.007 0.066 0.016
- added link pico_flexx_link_optical_frame
Joints:
- removed joint hokuyo_joint
- added joint pico_flexx_base_joint: type fixed, parent base_link, child pico_flexx_link_optical_frame, origin xyz=0.2 0 0.07 rpy=0 0 0
- added joint pico_flexx_depth_joint: type fixed, parent pico_flexx_link_optical_frame, child pico_flexx_depth_frame, origin xyz=0 0 0 rpy=${-M_PI/2} 0 ${-M_PI/2}
- added joint pico_flexx_joint: type fixed, parent pico_flexx_link_optical_frame, child pico_flexx_link, origin xyz=0 0 0 rpy=0 0 0
